File: stepper_controller_3x2.kicad_pcb (KiCad board)
At the start: 2 copper layers, 70.5 x 41.9 mm, 14 parts, among them P1 PWR_JACK_2.5x5.5, T1 TERM_BLK_HDR_4POS_VERT_0.2IN, T2 TERM_BLK_HDR_4POS_VERT_0.150IN, U1 TMC429, U2 MAX6817

Commit message: More progress towards v1.1.
Other:
- board text added: "2.5x5.5 Center + +12-30VDC"
- board text removed: "2.5x5.5 Center + +12-42VDC"
Changed lines of the file:
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@@
-(kicad_pcb (version 20170922) (host pcbnew no-vcs-found-9bd5522~60~ubuntu16.04.1)
+(kicad_pcb (version 20170922) (host pcbnew no-vcs-found-a562525~60~ubuntu16.04.1)
 (general
   (thickness 1.6)
@@
       (net 21 /tmc429_driver_0/REF_0) (solder_mask_margin 0.1016) (clearance 0.1016))
   )
-  (gr_text "2.5x5.5\nCenter +\n+12-42VDC" (at 149.86 98.425) (layer F.SilkS)
+  (gr_text "2.5x5.5\nCenter +\n+12-30VDC" (at 149.86 98.425) (layer F.SilkS)
     (effects (font (size 1.016 1.016) (thickness 0.254)))
   )
