File: stepper_controller_3x2.kicad_pcb (KiCad board)
At the start: 2 copper layers, 70.5 x 41.9 mm, 14 parts, among them P1 PWR_JACK_2.5x5.5, T1 TERM_BLK_HDR_4POS_VERT_0.2IN, T2 TERM_BLK_HDR_4POS_VERT_0.150IN, U1 TMC429, U2 MAX6817

Commit message: Finished version 1.1.
Parts:
- added C10: 470pF, stepper_controller_3x2:SM0805, B.Cu at (126.4, 75.6)
- added C11: 470pF, stepper_controller_3x2:SM0805, B.Cu at (123.8, 75.6)
- added C12: 0.1uF, stepper_controller_3x2:SM1210, B.Cu at (113.7, 84.5)
- added C6: 220uF_POL, stepper_controller_3x2:C_ELEC_10, F.Cu at (113.7, 95.2)
- added C7: 10uF, stepper_controller_3x2:SM1210, B.Cu at (122.6, 93.3)
- added C8: 470pF, stepper_controller_3x2:SM0805, B.Cu at (136.5, 75.6)
- added C9: 470pF, stepper_controller_3x2:SM0805, B.Cu at (134.0, 75.6)
- added L1: 90nH, stepper_controller_3x2:ECS-MPI4040, B.Cu at (137.8, 83.9)
- added L2: 90nH, stepper_controller_3x2:ECS-MPI4040, B.Cu at (132.7, 83.9)
- added L3: 90nH, stepper_controller_3x2:ECS-MPI4040, B.Cu at (127.6, 83.9)
- added L4: 90nH, stepper_controller_3x2:ECS-MPI4040, B.Cu at (122.6, 83.9)
- added R1: 1k, stepper_controller_3x2:SM1210, B.Cu at (99.7, 92.1)
- added REG1: CONV_DC_DC_5V_1A, stepper_controller_3x2:DC_DC_CONV_R78C, F.Cu at (99.1, 99.7)
- added RV1: VAR, stepper_controller_3x2:SM0805, B.Cu at (135.3, 78.1)
- added RV2: VAR, stepper_controller_3x2:SM0805, B.Cu at (125.1, 78.1)
- added RV3: VAR, stepper_controller_3x2:SM0805, B.Cu at (139.1, 75.6)
- added RV4: VAR, stepper_controller_3x2:SM0805, B.Cu at (131.4, 75.6)
- added RV5: VAR, stepper_controller_3x2:SM0805, B.Cu at (128.9, 75.6)
- added RV6: VAR, stepper_controller_3x2:SM0805, B.Cu at (121.3, 75.6)
- added U3: MAX6817, stepper_controller_3x2:MAX6817, B.Cu at (108.0, 84.5)
- C2: value 0.1uF -> 10uF
- C3: value 220uF_POL -> 10uF; footprint stepper_controller_3x2:C_ELEC_10 -> stepper_controller_3x2:SM1210; moved to B.Cu
- C4: value 10uF -> 0.1uF
- U2: value MAX6817 -> SN74ABT541BDWR; footprint stepper_controller_3x2:MAX6817 -> stepper_controller_3x2:SOIC_20
- moved D1 49.1 mm to (95.5, 75.1), turned to 90 degrees
- moved C4 35.2 mm to (88.9, 83.2), turned to 90 degrees
- moved C1 23.1 mm to (90.8, 89.5), turned to 0 degrees
- moved C5 19.0 mm to (118.1, 96.5), turned to 270 degrees
- moved CLK1 16.0 mm to (90.8, 94.6), turned to 0 degrees
- moved C3 14.0 mm to (99.7, 95.2), turned to 180 degrees
- moved C2 13.5 mm to (97.8, 102.9), turned to 0 degrees
- moved U2 11.5 mm to (109.2, 96.5), turned to 90 degrees
- moved U1 7.62 mm to (96.5, 85.1)
Connections:
- C2 pad 1: +3V3 -> VAA
- C3 pad 1: VDD -> +5V
- C4 pad 1: VDD -> +3V3
- C5 pad 1: +3V3 -> +5V
- MDB1 pad 23: (no net) -> +5V
- SS1 pad 15: +3V3 -> +5V
- SS1 pad 5: /CS_DRIVER_0 -> /tmc429_driver_0/~CS_DRIVER_0_B
- SS1 pad 6: /SCK -> /tmc429_driver_0/SCK_B
- SS1 pad 7: /MOSI -> /tmc429_driver_0/MOSI_B
- SS1 pad 8: /ENABLE_0 -> /tmc429_driver_0/~ENABLE_0_B
- SS1 pad 9: VDD -> VAA
- T1 pad 1: /tmc429_driver_0/stepper_0/B_- -> /tmc429_driver_0/stepper_0/B_-F
- T1 pad 2: /tmc429_driver_0/stepper_0/B_+ -> /tmc429_driver_0/stepper_0/B_+F
- T1 pad 3: /tmc429_driver_0/stepper_0/A_- -> /tmc429_driver_0/stepper_0/A_-F
- T1 pad 4: /tmc429_driver_0/stepper_0/A_+ -> /tmc429_driver_0/stepper_0/A_+F
- U2 pad 1: /tmc429_driver_0/stepper_0/REF_B -> GND
- U2 pad 2: GND -> /SCK
- U2 pad 3: /tmc429_driver_0/stepper_0/REFR_B -> /MOSI
- U2 pad 4: /tmc429_driver_0/REFR_0 -> /ENABLE_0
- U2 pad 5: +3V3 -> /CS_DRIVER_0
- U2 pad 6: /tmc429_driver_0/REF_0 -> GND
Routing:
- net GND: track 0.00 -> 233.4 mm
- net VAA: track 0.00 -> 108.3 mm
- net /MISO: track 0.00 -> 93.7 mm, vias 0 -> 1
- net +3V3: track 0.00 -> 87.0 mm, vias 0 -> 5
- net /tmc429_driver_0/DIR_0: track 0.00 -> 76.9 mm
- net /tmc429_driver_0/STEP_0: track 0.00 -> 72.4 mm
- net /ENABLE_0: track 0.00 -> 65.6 mm
- net /SCK: track 0.00 -> 60.4 mm, vias 0 -> 1
- net +5V: track 0.00 -> 60.2 mm, vias 0 -> 1
- net /MOSI: track 0.00 -> 53.5 mm
- net /tmc429_driver_0/REFR_0: track 0.00 -> 47.0 mm
- net /INT: track 0.00 -> 42.2 mm, vias 0 -> 1
- net /CS_429: track 0.00 -> 30.3 mm
- net /tmc429_driver_0/~CS_DRIVER_0_B: track 0.00 -> 29.6 mm
- net /tmc429_driver_0/SCK_B: track 0.00 -> 19.8 mm
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- added copper zone on B.Cu, net GND
- added copper zone on F.Cu, net VAA
Other:
- net class SUPERPOWER: trace_width 1.27 -> 1.0668
- board text added: "5V"
- board text added: "Disconnect Motor Driver Power Before Unplugging Motor Connectors"
- board text added: "Motor Driver Power 2.5x5.5 Center + +12-30VDC"
- board text removed: "2.5x5.5 Center + +12-30VDC"
