File: stepper_controller_3x2.kicad_pcb (KiCad board)
At the start: 2 copper layers, 70.5 x 41.9 mm, 34 parts, among them P1 PWR_JACK_2.5x5.5, T1 TERM_BLK_HDR_4POS_VERT_0.2IN, T2 TERM_BLK_HDR_4POS_VERT_0.150IN, U1 TMC429, U2 SN74ABT541BDWR, U3 MAX6817

Commit message: Progress towards v1.2
Parts:
- removed C10, C11: 470pF, stepper_controller_3x2:SM0805
- removed C12: 0.1uF, stepper_controller_3x2:SM1210
- removed L1, L2, L3, L4: 90nH, stepper_controller_3x2:ECS-MPI4040
- removed RV1, RV2, RV3, RV4, RV5, RV6: VAR, stepper_controller_3x2:SM0805
- added R2: 10.0k, footprints:SM0805, F.Cu at (126.4, 56.8)
- added R3: 845, stepper_controller_3x2:SM0805, F.Cu at (126.4, 59.7)
- added R4: 845, stepper_controller_3x2:SM0805, F.Cu at (130.6, 56.8)
- added R5: 845, stepper_controller_3x2:SM0805, F.Cu at (126.4, 62.6)
- added R6: 845, stepper_controller_3x2:SM0805, F.Cu at (130.6, 59.7)
- added U4: BUFFER_TRI_STATE, stepper_controller_3x2:SOT-23-5, F.Cu at (122.0, 61.8)
- added U5: OPTOISO_2CHAN, stepper_controller_3x2:SO-8, F.Cu at (116.4, 59.6)
- added U6: MAX6817, stepper_controller_3x2:MAX6817, F.Cu at (122.0, 58.0)
- C8, C9: value 470pF -> 0.1uF; footprint stepper_controller_3x2:SM0805 -> stepper_controller_3x2:SM1210
- R1: value 1k -> 10.0k; footprint stepper_controller_3x2:SM1210 -> footprints:SM0805
- U2: value SN74ABT541BDWR -> BUFFER_TRI_STATE; footprint stepper_controller_3x2:SOIC_20 -> stepper_controller_3x2:SOT-23-5
- U3: value MAX6817 -> SN74ABT541BDWR; footprint stepper_controller_3x2:MAX6817 -> stepper_controller_3x2:SOIC_20
- moved U1 61.0 mm to (97.8, 146.1)
- moved U3 41.0 mm to (121.3, 123.2)
- moved U2 40.5 mm to (139.1, 123.8)
- moved C7 35.1 mm to (149.2, 116.2)
- moved C9 29.5 mm to (157.5, 57.8)
- moved C5 28.0 mm to (139.7, 114.3)
- moved C2 27.4 mm to (72.4, 113.0)
- moved R1 25.3 mm to (88.9, 114.9)
- moved C3 20.8 mm to (104.1, 115.6)
- moved CLK1 19.6 mm to (73.7, 104.1)
- moved C8 19.0 mm to (144.8, 58.4)
- moved C1 15.3 mm to (76.2, 94.0)
- moved C4 13.4 mm to (75.6, 83.8)
Connections:
- C8 pad 1: /tmc429_driver_0/stepper_0/A_+F -> +3V3
- C9 pad 1: /tmc429_driver_0/stepper_0/A_-F -> +3V3
- MDB1 pad 23: +5V -> (no net)
- R1 pad 1: +5V -> +3V3
- R1 pad 2: GND -> /CS_429
- SS1 pad 4: /MISO -> /tmc429_driver_0/stepper_0/MISO_UB
- T1 pad 1: /tmc429_driver_0/stepper_0/B_-F -> /tmc429_driver_0/stepper_0/B_-
- T1 pad 2: /tmc429_driver_0/stepper_0/B_+F -> /tmc429_driver_0/stepper_0/B_+
- T1 pad 3: /tmc429_driver_0/stepper_0/A_-F -> /tmc429_driver_0/stepper_0/A_-
- T1 pad 4: /tmc429_driver_0/stepper_0/A_+F -> /tmc429_driver_0/stepper_0/A_+
- T2 pad 2: GND -> /tmc429_driver_0/stepper_0/REF_GND
- T2 pad 4: GND -> /tmc429_driver_0/stepper_0/REFR_GND
- U1 pad 1: +3V3 -> (no net)
- U1 pad 12: /MISO -> /tmc429_driver_0/MISO_UB
- U1 pad 13: +3V3 -> (no net)
- U1 pad 2: +3V3 -> (no net)
- U1 pad 29: +3V3 -> (no net)
- U2 pad 1: GND -> /CS_429
- U2 pad 2: /SCK -> /tmc429_driver_0/MISO_UB
- U2 pad 3: /MOSI -> GND
- U2 pad 4: /ENABLE_0 -> /MISO
- U2 pad 5: /CS_DRIVER_0 -> +3V3
- U3 pad 1: /tmc429_driver_0/stepper_0/REF_B -> GND
- U3 pad 2: GND -> /SCK
- U3 pad 3: /tmc429_driver_0/stepper_0/REFR_B -> /MOSI
- U3 pad 4: /tmc429_driver_0/REFR_0 -> /ENABLE_0
- U3 pad 5: +3V3 -> /CS_DRIVER_0
- U3 pad 6: /tmc429_driver_0/REF_0 -> GND
Routing:
- net GND: track 233.4 -> 218.3 mm
- net /tmc429_driver_0/stepper_0/A_-F: track 9.49 -> 0.00 mm
- net /tmc429_driver_0/stepper_0/B_+F: track 9.49 -> 0.00 mm
- net /tmc429_driver_0/stepper_0/B_+: track 3.83 -> 13.3 mm
- net /tmc429_driver_0/stepper_0/B_-F: track 9.49 -> 0.00 mm
- net /tmc429_driver_0/stepper_0/B_-: track 5.92 -> 15.4 mm
- net /tmc429_driver_0/stepper_0/A_+F: track 9.49 -> 0.00 mm
- net /ENABLE_0: track 65.6 -> 57.6 mm
- net /MOSI: track 53.5 -> 46.4 mm
- net /tmc429_driver_0/stepper_0/REF_B: track 6.66 -> 3.41 mm
- net /MISO: track 93.7 -> 91.9 mm
- net /tmc429_driver_0/stepper_0/REFR_B: track 3.64 -> 2.30 mm
- net +5V: track 60.2 -> 59.0 mm
Other:
- board text added: "Janelia Modular Device stepper_controller part_number: 1141 04/2019 ver 1.2 3x2"
- board text removed: "Janelia Modular Device stepper_controller part_number: 1141 10/2017 ver 1.1 3x2"

Commit message: Add limit switch filter capacitors
Parts:
- added C10: 0.1uF, stepper_controller_3x2:SM0805, B.Cu at (97.8, 87.6)
- added C11: 0.1uF, stepper_controller_3x2:SM0805, B.Cu at (94.6, 80.0)
- C1, C2, C3, C4, C5, C7, C8, C9: footprint stepper_controller_3x2:SM1210 -> stepper_controller_3x2:SM0805
- MDB1: value MODULAR_DEVICE_BASE_3X2_MALE -> VAL**
- R1: footprint footprints:SM0805 -> stepper_controller_3x2:SM0805
- R2: footprint footprints:SM0805 -> stepper_controller_3x2:SM0805; moved to B.Cu
- R3, R4, R5, R6, U4: moved to B.Cu
- U5: value OPTOISO_2CHAN -> VAL**; footprint stepper_controller_3x2:SO-8 -> stepper_controller_3x2:MAX6817; moved to B.Cu
- U6: value MAX6817 -> OPTOISO_2CHAN; footprint stepper_controller_3x2:MAX6817 -> stepper_controller_3x2:SO-8; moved to B.Cu
- moved C9 63.9 mm to (101.0, 87.6), turned to 270 degrees
- moved U2 59.2 mm to (89.5, 91.4), turned to 180 degrees
- moved U3 54.8 mm to (146.1, 74.3), turned to 90 degrees
- moved C8 50.0 mm to (104.1, 87.6), turned to 270 degrees
- moved U1 49.7 mm to (106.7, 97.2)
- moved C5 42.6 mm to (154.3, 74.3)
- moved CLK1 42.4 mm to (115.6, 97.8), turned to 180 degrees
- moved C1 39.4 mm to (115.6, 92.1), turned to 180 degrees
- moved C7 36.0 mm to (122.6, 92.1)
- moved R2 35.4 mm to (130.2, 92.1)
- moved U4 35.0 mm to (130.2, 95.9), turned to 180 degrees
- moved R3 33.7 mm to (102.2, 83.2)
- moved R4 31.3 mm to (106.0, 76.2), turned to 90 degrees
- moved U6 31.1 mm to (108.0, 85.7)
- moved C4 27.9 mm to (101.0, 95.2)
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Connections:
- C9 pad 1: +3V3 -> /tmc429_driver_0/stepper_0/REF_BI
- U1 pad 1: (no net) -> +3V3
- U1 pad 13: (no net) -> +3V3
- U1 pad 2: (no net) -> +3V3
- U1 pad 29: (no net) -> +3V3
- U1 pad 7: /CS_429 -> /tmc429_driver_0/~CS
- U2 pad 1: /CS_429 -> /tmc429_driver_0/~CS
- U5 pad 1: /tmc429_driver_0/stepper_0/REF_PWR -> /tmc429_driver_0/stepper_0/REF_BI
- U5 pad 2: /tmc429_driver_0/stepper_0/REF_B -> GND
- U5 pad 3: /tmc429_driver_0/stepper_0/REFR_B -> /tmc429_driver_0/stepper_0/REFR_BI
- U5 pad 4: /tmc429_driver_0/stepper_0/REFR_PWR -> /tmc429_driver_0/REFR_0
- U5 pad 5: GND -> +3V3
- U5 pad 6: /tmc429_driver_0/stepper_0/REFR_BI -> /tmc429_driver_0/REF_0
- U6 pad 1: /tmc429_driver_0/stepper_0/REF_BI -> /tmc429_driver_0/stepper_0/REF_PWR
- U6 pad 2: GND -> /tmc429_driver_0/stepper_0/REF_B
- U6 pad 3: /tmc429_driver_0/stepper_0/REFR_BI -> /tmc429_driver_0/stepper_0/REFR_B
- U6 pad 4: /tmc429_driver_0/REFR_0 -> /tmc429_driver_0/stepper_0/REFR_PWR
- U6 pad 5: +3V3 -> GND
- U6 pad 6: /tmc429_driver_0/REF_0 -> /tmc429_driver_0/stepper_0/REFR_BI
Routing:
- net /MOSI: track 46.4 -> 136.4 mm
- net +5V: track 59.0 -> 124.3 mm, vias 1 -> 3
- net /CS_DRIVER_0: track 14.9 -> 66.5 mm, vias 0 -> 1
- net /tmc429_driver_0/SCK_B: track 19.8 -> 61.2 mm, vias 0 -> 1
- net /tmc429_driver_0/MOSI_B: track 18.5 -> 59.2 mm, vias 0 -> 1
- net +3V3: track 87.0 -> 125.6 mm, vias 5 -> 3
- net /tmc429_driver_0/~ENABLE_0_B: track 17.8 -> 54.3 mm, vias 0 -> 1
- net /tmc429_driver_0/STEP_0: track 72.4 -> 35.9 mm, vias 0 -> 1
- net /tmc429_driver_0/MISO_UB: track 0.00 -> 36.5 mm
- net /tmc429_driver_0/DIR_0: track 76.9 -> 40.6 mm, vias 0 -> 1
- net /tmc429_driver_0/~CS_DRIVER_0_B: track 29.6 -> 61.1 mm
- net /tmc429_driver_0/stepper_0/REFR_BI: track 0.00 -> 24.6 mm
- net /tmc429_driver_0/~CS: track 0.00 -> 24.0 mm, vias 0 -> 2
- net VAA: track 108.3 -> 85.3 mm, vias 0 -> 1
- net /CS_429: track 30.3 -> 53.2 mm
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- added copper zone on F.Cu, net GND
- added copper zone on B.Cu, net VAA
- removed copper zone on B.Cu, net GND
- removed copper zone on F.Cu, net VAA
